Commit message: copy from https://github.com/TixiaoShan/LIO-SAM 4fc42fabd94da4c1b7778291627a07f7d841aa98 and fix for ROS noetic, opencv2, flann compile error.

File: launch/include/config/robot.urdf.xacro (robot description, xacro)
@@ -21,8 +21,8 @@
     <origin xyz="0 0 0" rpy="0 0 0" />
   </joint>
-  <link name="rtk"> </link>
+  <link name="navsat_link"> </link>
   <joint name="navsat_joint" type="fixed">
     <parent link="chassis_link" />
-    <child link="rtk" />
+    <child link="navsat_link" />
     <origin xyz="0 0 0" rpy="0 0 0" />
   </joint>
